File: PacMan.kicad_pcb (KiCad board)
At the start: 2 copper layers, 135.9 x 127 mm, 126 parts, among them J1 POWER+, J12 CHRG TEST, J13 AIR Left, J14 AIR Right, J2 POWER-, J3 TSV IN, J4 Charge Detection, J5 CellMen, J6 RJ12, J7 Panel, J8 SLOOP, J9 GLV/CAN, K1 G5Q-1A4 DC24, K2 T9AS1D12-48, K3 T9AS1D12-48, Q1 BSS123, Q2 DMP10H4D2S, Q3 BSS123, Q4 DMP10H4D2S, U1 MCP9804, U10 LTC4151, U11 INA592, U12 PDQE10-Q24-S9-D, U13 V7805-500, U14 L78L05_SOT89, U15 Si8605AD-B-IS, U2 TEC2-4815WI, U3 ADM6320, U4 MCP2551-I-SN, U5 ESP32_TTGO_PSRAM, U6 MCP23008, U7 RTC, U8 ACHS-7122, U9 PDQE10-Q48-S24-D

Commit message: Updated some power stuff
Parts:
- removed C24, C25: 0.1u/50V, Capacitor_SMD:C_0805_2012Metric_Pad1.15x1.40mm_HandSolder
- removed J12: CHRG TEST, Connector_PinHeader_2.54mm:PinHeader_1x02_P2.54mm_Vertical
- removed R31: 500k, Resistor_SMD:R_0805_2012Metric_Pad1.15x1.40mm_HandSolder
- removed R33, R34, R36, R37: 4.7k, Resistor_SMD:R_0805_2012Metric_Pad1.15x1.40mm_HandSolder
- added R27: 4.7k, Resistor_SMD:R_0805_2012Metric_Pad1.15x1.40mm_HandSolder, F.Cu at (138.2, 121.3)
- added U16: TEC3-2419, Lafayette_Electric_Car_Footprints:TEC2-4815, F.Cu at (163.8, 32.4)
- added U17: TEC3-2419, Lafayette_Electric_Car_Footprints:TEC2-4815, F.Cu at (149.2, 32.4)
- C10, C11, C14, C15, C18, C19, C7, C8, C9, TP8, TP9: moved to F.Cu
- C17: value 22u/50V -> 0.1u/50V; moved to F.Cu
- C20: value 10u/50V -> 0.1u/50V; footprint Capacitor_SMD:C_1210_3225Metric_Pad1.42x2.65mm_HandSolder -> Capacitor_SMD:C_0805_2012Metric_Pad1.15x1.40mm_HandSolder; moved to F.Cu
- C21: value 0.33u/50V -> 0.1u/50V
- K2, K3: value T9AS1D12-48 -> T9AS1D12-24
- Q2: value DMP10H4D2S -> 2N7002; footprint Package_TO_SOT_SMD:SOT-23_Handsoldering -> Package_TO_SOT_SMD:SOT-23
- R19: value 15k -> 4.7k
- R20, R21: value 560 -> 4.7k
- R22: value 1k -> 4.7k
- R23: value 390 -> 4.7k
- U12: value PDQE10-Q24-S9-D -> VIFSD1-S24-S5-SIP; footprint Lafayette_Electric_Car_Footprints:PDQE10-DIP6 -> Lafayette_Electric_Car_Footprints:VIFSD1-S24-S5-SIP
- U14: value L78L05_SOT89 -> Si8600AC; footprint Package_TO_SOT_SMD:SOT-89-3_Handsoldering -> Package_SO:SO-8_3.9x4.9mm_P1.27mm; moved to B.Cu
- U15: value Si8605AD-B-IS -> Si8600AC; footprint Package_SO:SOIC-16W_7.5x10.3mm_P1.27mm -> Package_SO:SO-8_3.9x4.9mm_P1.27mm; moved to B.Cu
- moved ISO4 208.6 mm to (302.9, 23.5)
- moved K1 163.3 mm to (45.8, 27.6), turned to 0 degrees
- moved D1 162.5 mm to (22.3, 73.4), turned to 0 degrees
- moved J7 158.5 mm to (21.5, 98.1)
- moved ISO2 148.5 mm to (306.1, 23.5)
- moved U6 147.1 mm to (50.2, 33.0), turned to 0 degrees
- moved R40 142.8 mm to (67.7, 35.4)
- moved Q1 142.8 mm to (58.0, 40.2)
- moved R39 140.9 mm to (87.1, 18.1)
- moved ISO5 138.6 mm to (60.4, 30.4)
- moved U5 137.9 mm to (19.4, 23.3), turned to 0 degrees
- moved R3 137.8 mm to (68.4, 44.3)
- moved ISO6 137.3 mm to (49.9, 39.5)
- moved C6 134.4 mm to (54.8, 49.9)
- moved H2 132.0 mm to (65.5, 98.6)
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Connections:
- C17 pad 1: /LV_24V -> /Isolation/SEG1_5V
- C17 pad 2: /GLV_RTN -> /Isolation/SEG1_RTN
- C20 pad 1: /TSV_9V -> /Isolation/SEG2_5V
- C20 pad 2: /PACK_RTN -> /Isolation/SEG2_RTN
- C21 pad 1: /TSV_9V -> /LV_5V
- C21 pad 2: /PACK_RTN -> /GLV_RTN
- C22 pad 1: /TSV_5V -> /LV_5V
- C22 pad 2: /PACK_RTN -> /GLV_RTN
- D4 pad 1: Net-(D4-Pad1) -> /Charging/LV_24V
- D4 pad 2: /CHRG_IN- -> Net-(D4-Pad2)
- ISO2 pad 1: Net-(ISO2-Pad1) -> (no net)
- ISO2 pad 2: /GLV_RTN -> Net-(C23-Pad1)
- ISO2 pad 3: /CHRG_IN- -> (no net)
- ISO2 pad 4: /Charging/EN_CHRG_ISO -> (no net)
- K2 pad 1: Net-(D4-Pad1) -> /Charging/LV_24V
- K2 pad 2: /CHRG_IN- -> Net-(D4-Pad2)
- K2 pad 3: /Charging/CurrentSensor+ -> /CHRG_IN+
- K2 pad 4: /CHRG_IN+ -> /Charging/CurrentSensor+
- K3 pad 1: Net-(D4-Pad1) -> /Charging/LV_24V
- K3 pad 2: /CHRG_IN- -> Net-(D4-Pad2)
- K3 pad 3: /PACK- -> /CHRG_IN-
- K3 pad 4: /CHRG_IN- -> /PACK-
- Q2 pad 1: /Charging/EN_CHRG_ISO -> /CHRG_EN
- Q2 pad 2: Net-(Q2-Pad2) -> /GLV_RTN
- Q2 pad 3: /CHRG_IN+ -> Net-(D4-Pad2)
- R19 pad 1: Net-(J12-Pad2) -> /Isolation/SEG1_5V
- R19 pad 2: /CHRG_IN- -> /Isolation/SDA_SEG1
- R20 pad 1: Net-(D4-Pad1) -> /Isolation/SEG2_5V
- R20 pad 2: Net-(Q2-Pad2) -> /Isolation/SDA_SEG2
- R21 pad 1: Net-(Q2-Pad2) -> /Isolation/SEG1_5V
- R21 pad 2: Net-(D4-Pad1) -> /Isolation/SCL_SEG1
- R22 pad 1: /CHRG_IN+ -> /Isolation/SEG2_5V
- R22 pad 2: /Charging/EN_CHRG_ISO -> /Isolation/SCL_SEG2
- R23 pad 1: /CHRG_EN -> /LV_5V
- R23 pad 2: Net-(ISO2-Pad1) -> /SDA_GLV
- U10 pad 1: /PACK_FUSED -> Net-(U10-Pad1)
- U10 pad 10: /Power/PACK_FUSED_CS -> (no net)
- U10 pad 2: /PACK_FUSED -> Net-(U10-Pad1)
- U12 pad 1: /GLV_RTN -> /LV_24V
- U12 pad 2: /LV_24V -> /GLV_RTN
- U14 pad 1: /TSV_5V -> /LV_5V
- U14 pad 2: /PACK_RTN -> /SDA_GLV
- U14 pad 3: /TSV_9V -> /SCL_GLV
- U15 pad 1: /TSV_5V -> /LV_5V
- U15 pad 2: (no net) -> /SDA_GLV
- U15 pad 3: /SDA_TSV -> /SCL_GLV
- U15 pad 4: Net-(C23-Pad1) -> /GLV_RTN
- U15 pad 5: (no net) -> /Isolation/SEG2_RTN
- U15 pad 6: /SCL_TSV -> /Isolation/SCL_SEG2
- U15 pad 7: (no net) -> /Isolation/SDA_SEG2
- U15 pad 8: /PACK_RTN -> /Isolation/SEG2_5V
- U5 pad 23: /~CHRG_DETECT -> (no net)
Routing:
- net /LV_5V: track 278.0 -> 0.00 mm, vias 8 -> 0
- net /LV_24V: track 251.8 -> 0.00 mm
- net /LV_3V3: track 193.4 -> 0.00 mm, vias 15 -> 0
- net /GLV_24V: track 174.3 -> 0.00 mm
- net /SCL_GLV: track 168.5 -> 0.00 mm, vias 6 -> 0
- net /SDA_GLV: track 162.9 -> 0.00 mm, vias 6 -> 0
- net /CHS_GND: track 142.2 -> 0.00 mm
- net /AIRS-: track 140.8 -> 0.00 mm, vias 2 -> 0
- net /CHRG_IN-: track 130.2 -> 0.00 mm
- net /TSV_5V: track 127.9 -> 0.00 mm, vias 8 -> 0
- net /GLV_RTN: track 120.9 -> 0.00 mm, vias 25 -> 0
- net /AIRS+: track 115.9 -> 0.00 mm, vias 2 -> 0
- net /TSV_9V: track 114.0 -> 0.00 mm
- net /DISP_RST: track 111.2 -> 0.00 mm, vias 7 -> 0
- net /MCU/~RESET: track 86.7 -> 0.00 mm, vias 2 -> 0
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- removed copper zone on F.Cu, net (none)
- removed copper zone on B.Cu, net /CHRG_IN+
- removed copper zone on F.Cu, net /CHRG_IN+
- removed copper zone on B.Cu, net /CHRG_IN-
- removed copper zone on F.Cu, net /CHRG_IN-
- removed copper zone on B.Cu, net /Charging/CurrentSensor+
- removed copper zone on F.Cu, net /Charging/CurrentSensor+
- removed copper zone on B.Cu, net /GLV_RTN
- removed copper zone on B.Cu, net /PACK+
- removed copper zone on F.Cu, net /PACK+
- removed copper zone on B.Cu, net /PACK-
- removed copper zone on F.Cu, net /PACK-
- removed copper zone on B.Cu, net /PACK_RTN
- removed copper zone on F.Cu, net /PACK_RTN
Other:
- board outline removed
- board text removed: "AIRS"
- board text removed: "Accumulator Management System Fall 2019"
- board text removed: "Bus Bar Current Sensor"
- board text removed: "Danger! High Voltage!"
- board text removed: "GLV"
- board text removed: "LED1"
- board text removed: "LED2"
- board text removed: "Made in USA!"
- board text removed: "PacMan v1.0 - Jon Abel"
- board text removed: "S/N"
- board text removed: "TSV!"

Commit message: Started work on new layout
Parts:
- added C24: 4.7uF/50V, Capacitor_SMD:C_0805_2012Metric_Pad1.15x1.40mm_HandSolder, F.Cu at (-59.4, 111.8)
- added C25: 4.7uF/50V, Capacitor_SMD:C_0805_2012Metric_Pad1.15x1.40mm_HandSolder, B.Cu at (106.0, 95.5)
- added C26: 4.7uF/50V, Capacitor_SMD:C_0805_2012Metric_Pad1.15x1.40mm_HandSolder, B.Cu at (89.5, 95.5)
- added C27: 4.7uF, Capacitor_SMD:C_0805_2012Metric_Pad1.15x1.40mm_HandSolder, F.Cu at (-64.2, 111.8)
- added C28: 10u, Capacitor_SMD:C_1210_3225Metric_Pad1.42x2.65mm_HandSolder, B.Cu at (105.4, 82.5)
- added C29: 10u, Capacitor_SMD:C_1210_3225Metric_Pad1.42x2.65mm_HandSolder, B.Cu at (88.9, 82.5)
- added C31: 1u, Capacitor_SMD:C_0805_2012Metric_Pad1.15x1.40mm_HandSolder, F.Cu at (100.3, 77.5)
- added C33: 2.2u, Capacitor_SMD:C_0805_2012Metric_Pad1.15x1.40mm_HandSolder, F.Cu at (100.3, 83.8)
- added J10: SEG2 CellMen, Connector_IDC:IDC-Header_2x03_P2.54mm_Vertical, F.Cu at (92.1, 62.2)
- added Q5: DMP10H4D2S, Package_TO_SOT_SMD:SOT-23, F.Cu at (222.9, 76.2)
- added R28: 100k, Resistor_SMD:R_0805_2012Metric_Pad1.15x1.40mm_HandSolder, F.Cu at (222.9, 73.0)
- added R31: R, Resistor_SMD:R_0805_2012Metric_Pad1.15x1.40mm_HandSolder, B.Cu at (217.2, 81.9)
- added R33: 10k, Resistor_SMD:R_0805_2012Metric_Pad1.15x1.40mm_HandSolder, F.Cu at (-99.1, 113.8)
- added TP10: SEG1_5V, Resistor_SMD:R_0805_2012Metric_Pad1.15x1.40mm_HandSolder, F.Cu at (-59.4, 114.8)
- added TP11: SEG1_RTN, Resistor_SMD:R_0805_2012Metric_Pad1.15x1.40mm_HandSolder, F.Cu at (-59.4, 117.7)
- added TP12: SEG2_9V, TestPoint:TestPoint_Pad_D2.0mm, F.Cu at (-63.1, 121.2)
- added TP13: SEG2_5V, TestPoint:TestPoint_Pad_D2.0mm, F.Cu at (-48.9, 107.7)
- added TP14: SEG2_RTN, TestPoint:TestPoint_Pad_D2.0mm, F.Cu at (-55.0, 115.3)
- added U18: AP2204K-5.0, Package_TO_SOT_SMD:SOT-23-5, F.Cu at (100.3, 80.6)
- added U20: Si8600AC, Package_SO:SO-8_3.9x4.9mm_P1.27mm, F.Cu at (-97.2, 109.1)
- D4, ISO2, ISO4: moved to B.Cu
- J5: value CellMen -> SEG1 CellMen
- Q2: footprint Package_TO_SOT_SMD:SOT-23 -> Package_TO_SOT_SMD:SOT-23_Handsoldering; moved to B.Cu
- TP3: value TSV_9V -> SEG1_9V; footprint TestPoint:TestPoint_Pad_D2.0mm -> Resistor_SMD:R_0805_2012Metric_Pad1.15x1.40mm_HandSolder
- U16, U17: footprint Lafayette_Electric_Car_Footprints:TEC2-4815 -> Lafayette_Electric_Car_Footprints:TEC3-2419
- moved C15 232.4 mm to (-90.6, 103.8)
- moved C19 232.4 mm to (-92.9, 99.5)
- moved TP2 232.4 mm to (-75.6, 98.3)
- moved TP4 232.4 mm to (-85.3, 102.3)
- moved TP5 232.4 mm to (-80.9, 100.1)
- moved TP7 232.4 mm to (-75.6, 94.2)
- moved C16 232.4 mm to (-80.0, 93.7)
- moved C18 232.4 mm to (-79.4, 90.1)
- moved TP1 232.4 mm to (-80.0, 96.6)
- moved TP6 232.4 mm to (-68.4, 86.5)
- moved C14 232.4 mm to (-74.1, 89.5)
- moved R26 232.4 mm to (-72.8, 85.9)
- moved TP3 211.1 mm to (-64.2, 114.8)
- moved C17 201.3 mm to (-78.8, 113.4)
- moved C20 201.3 mm to (-88.3, 113.8)
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Connections:
- net /Isolation/SCL_SEG2 renamed /SCL_SEG2
- net /Isolation/SDA_SEG2 renamed /SDA_SEG2
- net /Isolation/SEG1_5V renamed /SEG1_5V
- net /Isolation/SEG2_5V renamed /SEG2_5V
- C17 pad 2: /Isolation/SEG1_RTN -> /SEG1_RTN
- C20 pad 2: /Isolation/SEG2_RTN -> /SEG2_RTN
- D4 pad 1: /Charging/LV_24V -> /LV_24V
- ISO2 pad 1: (no net) -> Net-(ISO2-Pad1)
- ISO2 pad 2: Net-(C23-Pad1) -> Net-(ISO2-Pad2)
- ISO2 pad 3: (no net) -> /GLV_RTN
- ISO2 pad 4: (no net) -> /~CHRG_DETECT
- J3 pad 1: /TSV_VEHICLE+ -> /TSV_VEHICLE-
- J3 pad 2: /TSV_VEHICLE- -> /TSV_VEHICLE+
- J5 pad 1: /SDA_TSV -> /SEG1_9V
- J5 pad 2: /SCL_TSV -> /SEG1_RTN
- J5 pad 3: /TSV_9V -> /SCL_SEG1
- J5 pad 4: /PACK_RTN -> /SDA_SEG1
- J5 pad 5: (no net) -> /SEG1_RTN
- J5 pad 6: (no net) -> /SEG1_9V
- K2 pad 1: /Charging/LV_24V -> /LV_24V
- K2 pad 3: /CHRG_IN+ -> /Charging/CurrentSensor+
- K2 pad 4: /Charging/CurrentSensor+ -> /CHRG_IN+
- K3 pad 1: /Charging/LV_24V -> /LV_24V
- K3 pad 3: /CHRG_IN- -> /PACK-
- K3 pad 4: /PACK- -> /CHRG_IN-
- R19 pad 2: /Isolation/SDA_SEG1 -> /SDA_SEG1
- R21 pad 2: /Isolation/SCL_SEG1 -> /SCL_SEG1
- TP3 pad 1: /TSV_9V -> /SEG1_9V
- U10 pad 1: Net-(U10-Pad1) -> /PACK_FUSED
- U10 pad 10: (no net) -> /Power/PACK_FUSED_CS
- U10 pad 2: Net-(U10-Pad1) -> /PACK_FUSED
- U10 pad 6: /SCL_TSV -> /SCL_SEG1
- U10 pad 7: /SDA_TSV -> /SDA_SEG1
- U12 pad 4: (no net) -> /PACK_RTN
- U12 pad 6: (no net) -> /TSV_5V
- U14 pad 5: /Isolation/SEG1_RTN -> /SEG1_RTN
- U14 pad 6: /Isolation/SCL_SEG1 -> /SCL_SEG1
- U14 pad 7: /Isolation/SDA_SEG1 -> /SDA_SEG1
- U15 pad 5: /Isolation/SEG2_RTN -> /SEG2_RTN
- U16 pad 6: (no net) -> /SEG1_9V
- U16 pad 7: (no net) -> /SEG1_RTN
- U17 pad 6: (no net) -> /SEG2_9V
- U17 pad 7: (no net) -> /SEG2_RTN
- U5 pad 23: (no net) -> /~CHRG_DETECT
Routing:
- net Net-(ISO2-Pad1): track 0.00 -> 14.0 mm, vias 0 -> 1
- net Net-(C23-Pad1): track 0.00 -> 6.67 mm
- net /SEG2_9V: track 0.00 -> 4.95 mm
- net /SEG2_RTN: track 0.00 -> 3.27 mm
- net /TSV_5V: track 0.00 -> 3.19 mm
- added copper zone on F.Cu, net /CHRG_IN+
- added copper zone on F.Cu, net /CHRG_IN-
- added copper zone on F.Cu, net /Charging/CurrentSensor+
- added copper zone on F.Cu, net /PACK+
- added copper zone on F.Cu, net /PACK-
Other:
- board outline added: 139.7 x 127 mm
- net class TSV Pre Fuse added: clearance 3.2, trace_width 5, via_dia 0.8, via_drill 0.4

Commit message: quick change
Parts:
- removed C31: 1u, Capacitor_SMD:C_0805_2012Metric_Pad1.15x1.40mm_HandSolder
- removed C33: 2.2u, Capacitor_SMD:C_0805_2012Metric_Pad1.15x1.40mm_HandSolder
- removed U20: Si8600AC, Package_SO:SO-8_3.9x4.9mm_P1.27mm
- added C30: 1u, Capacitor_SMD:C_0805_2012Metric_Pad1.15x1.40mm_HandSolder, F.Cu at (97.8, 76.8)
- added C32: 2.2u, Capacitor_SMD:C_0805_2012Metric_Pad1.15x1.40mm_HandSolder, F.Cu at (102.5, 76.8)
- C10, C11, C15, C24, C27, C7, C8, C9: moved to B.Cu
- moved R33 315.8 mm to (216.1, 95.2)
- moved R18 280.0 mm to (209.6, 109.2), turned to 180 degrees
- moved R12 278.3 mm to (209.6, 120.7), turned to 180 degrees
- moved C11 274.9 mm to (209.6, 111.1)
- moved R10 273.9 mm to (209.6, 124.5), turned to 180 degrees
- moved C7 272.9 mm to (209.6, 126.4)
- moved R16 270.7 mm to (209.6, 113.0), turned to 180 degrees
- moved C10 270.3 mm to (209.6, 114.9)
- moved R9 268.7 mm to (209.6, 126.4), turned to 180 degrees
- moved R17 265.0 mm to (209.6, 111.1), turned to 180 degrees
- moved R15 263.0 mm to (209.6, 114.9), turned to 180 degrees
- moved C8 260.4 mm to (209.6, 122.6)
- moved C9 260.0 mm to (209.6, 118.7)
- moved R13 257.8 mm to (209.6, 118.7), turned to 180 degrees
- moved R11 256.0 mm to (209.6, 122.6), turned to 180 degrees
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Routing:
- net /LV_3V3: track 0.00 -> 22.8 mm, vias 0 -> 5
- net /MCU/BTN_UP_MCU: track 0.00 -> 4.94 mm, vias 0 -> 1
- net /MCU/BTN_RIGHT_MCU: track 0.00 -> 4.94 mm, vias 0 -> 1
- net /MCU/BTN_LEFT_MCU: track 0.00 -> 4.94 mm, vias 0 -> 1
- net /MCU/BTN_DOWN_MCU: track 0.00 -> 4.94 mm, vias 0 -> 1
- net /MCU/BTN_CENTER_MCU: track 0.00 -> 4.94 mm, vias 0 -> 1

Commit message: Added connectors for cell balancing, made big progress on new layout
Parts:
- removed TP1: TSV_RTN, Resistor_SMD:R_0805_2012Metric_Pad1.15x1.40mm_HandSolder
- removed TP10: SEG1_5V, Resistor_SMD:R_0805_2012Metric_Pad1.15x1.40mm_HandSolder
- removed TP11: SEG1_RTN, Resistor_SMD:R_0805_2012Metric_Pad1.15x1.40mm_HandSolder
- removed TP2: TSV_5V, TestPoint:TestPoint_Pad_D2.0mm
- removed TP3: SEG1_9V, Resistor_SMD:R_0805_2012Metric_Pad1.15x1.40mm_HandSolder
- removed TP4: LV_RTN, Resistor_SMD:R_0805_2012Metric_Pad1.15x1.40mm_HandSolder
- removed TP5: LV_5V, TestPoint:TestPoint_Pad_D2.0mm
- removed TP6: LV_24V, TestPoint:TestPoint_Pad_D2.0mm
- removed TP7: GLV_24V, TestPoint:TestPoint_Pad_D2.0mm
- removed TP8: SDA, TestPoint:TestPoint_Pad_D2.0mm
- removed TP9: SCL, TestPoint:TestPoint_Pad_D2.0mm
- added J11: SEG1 Balance, Lafayette_Electric_Car_Footprints:Molex_Mini-Fit_Jr_5566-02A_2x01_P4.20mm_Vertical, F.Cu at (130.8, 45.7)
- added J12: SEG2 Balance, Lafayette_Electric_Car_Footprints:Molex_Mini-Fit_Jr_5566-02A_2x01_P4.20mm_Vertical, F.Cu at (114.9, 41.7)
- added J15: SEG1, Lafayette_Electric_Car_Footprints:Molex_Mini-Fit_Jr_5566-02A_2x01_P4.20mm_Vertical, F.Cu at (123.8, 45.7)
- added J16: SEG2, Lafayette_Electric_Car_Footprints:Molex_Mini-Fit_Jr_5566-02A_2x01_P4.20mm_Vertical, F.Cu at (107.8, 41.7)
- C14, C17, C18, C19, C20, C21, C22, R23, R27, R33, R35: moved to B.Cu
- J6: value RJ12 -> BusBar Current Sensor
- J8: footprint Lafayette_Electric_Car_Footprints:Molex_Mini-Fit_Jr_5566-08A2_2x04_P4.20mm_Vertical -> Connector_Molex:Molex_Mini-Fit_Jr_5566-08A_2x04_P4.20mm_Vertical
- J9: footprint Lafayette_Electric_Car_Footprints:Molex_Mini-Fit_Jr_5566-12A2_2x06_P4.20mm_Vertical -> Connector_Molex:Molex_Mini-Fit_Jr_5566-12A_2x06_P4.20mm_Vertical
- Q1, Q3, Q4: footprint Package_TO_SOT_SMD:SOT-23_Handsoldering -> Package_TO_SOT_SMD:SOT-23
- Q2: footprint Package_TO_SOT_SMD:SOT-23_Handsoldering -> Package_TO_SOT_SMD:SOT-23; moved to F.Cu
- moved R23 273.0 mm to (163.2, 110.5), turned to 90 degrees
- moved R27 270.6 mm to (160.7, 110.5), turned to 90 degrees
- moved R39 257.2 mm to (210.2, 146.1), turned to 270 degrees
- moved ISO5 256.0 mm to (204.5, 146.1)
- moved ISO6 255.6 mm to (204.5, 141.6)
- moved ISO1 255.1 mm to (204.5, 137.2)
- moved R40 250.5 mm to (210.2, 141.6), turned to 270 degrees
- moved R38 249.8 mm to (198.8, 141.6), turned to 270 degrees
- moved R3 249.2 mm to (210.2, 137.2), turned to 270 degrees
- moved R5 244.6 mm to (198.8, 146.1), turned to 270 degrees
- moved R2 243.3 mm to (198.8, 137.2), turned to 270 degrees
- moved R19 220.8 mm to (113.0, 74.9), turned to 180 degrees
- moved R21 217.6 mm to (108.8, 74.9)
- moved U6 217.6 mm to (196.8, 117.5)
- moved R20 214.2 mm to (97.2, 71.1), turned to 180 degrees
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Connections:
- C1 pad 1: /LV_5V -> /LV_3V3
- C21 pad 1: /LV_5V -> /LV_3V3
- C22 pad 1: /LV_5V -> /LV_3V3
- C30 pad 1: /SEG1_9V -> /SEG2_9V
- C30 pad 2: /SEG1_RTN -> /SEG2_RTN
- C32 pad 1: /SEG1_5V -> /SEG2_5V
- C32 pad 2: /SEG1_RTN -> /SEG2_RTN
- C6 pad 1: /LV_5V -> /LV_3V3
- J7 pad 10: /DISP_RST -> /DISP_CLK
- J7 pad 11: /DISP_CS -> /DISP_BUSY
- J7 pad 13: /DISP_DIN -> /DISP_DC
- J7 pad 15: /DISP_CLK -> /DISP_RST
- J7 pad 17: /DISP_DC -> /DISP_CS
- J7 pad 19: /DISP_BUSY -> /DISP_DIN
- J7 pad 4: /TSV_LIVE -> /LV_24V
- J7 pad 6: /LV_24V -> /TSV_LIVE
- K1 pad 3: /SLOOP1_IN -> /SLOOP1_OUT
- K1 pad 4: /SLOOP1_OUT -> /SLOOP1_IN
- R23 pad 1: /LV_5V -> /LV_3V3
- R27 pad 1: /LV_5V -> /LV_3V3
- R33 pad 2: /LV_5V -> /LV_3V3
- U1 pad 8: /LV_5V -> /LV_3V3
- U14 pad 1: /LV_5V -> /LV_3V3
- U15 pad 1: /LV_5V -> /LV_3V3
- U18 pad 1: /SEG1_9V -> /SEG2_9V
- U18 pad 2: /SEG1_RTN -> /SEG2_RTN
- U18 pad 3: /SEG1_9V -> /SEG2_9V
- U18 pad 5: /SEG1_5V -> /SEG2_5V
- U5 pad 17: /CHRG_EN -> /~CHRG_DETECT
- U5 pad 22: /SDA_GLV -> /CHRG_EN
- U5 pad 23: /~CHRG_DETECT -> /SDA_GLV
- U6 pad 20: /LV_5V -> /LV_3V3
Routing:
- net /LV_24V: track 0.00 -> 190.1 mm, vias 0 -> 4
- net /GLV_24V: track 0.00 -> 144.3 mm
- net /AIRS-: track 0.00 -> 136.3 mm, vias 0 -> 5
- net /LV_5V: track 0.00 -> 134.8 mm, vias 0 -> 2
- net /SDA_GLV: track 0.00 -> 124.9 mm, vias 0 -> 4
- net /SCL_GLV: track 0.00 -> 119.7 mm, vias 0 -> 4
- net /AIRS+: track 0.00 -> 118.3 mm, vias 0 -> 5
- net /LV_3V3: track 22.8 -> 129.9 mm, vias 5 -> 6
- net /DISP_RST: track 0.00 -> 90.9 mm, vias 0 -> 5
- net /DISP_DC: track 0.00 -> 83.8 mm, vias 0 -> 4
- net /MCU/WATCHDOG: track 0.00 -> 80.3 mm, vias 0 -> 5
- net /MCU/BTN_LEFT_MCU: track 4.94 -> 80.4 mm
- net /DISP_BUSY: track 0.00 -> 74.9 mm, vias 0 -> 3
- net /SEG2_9V: track 4.95 -> 76.9 mm, vias 0 -> 3
- net /DISP_CLK: track 0.00 -> 70.8 mm
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- added copper zone on B.Cu, net /GLV_RTN
- added copper zone on F.Cu, net /PACK_RTN
- added copper zone on B.Cu, net /SEG2_RTN
Other:
- board size 139.7 x 127 mm -> 140.3 x 141.6 mm
- board text added: "GREEN"
- board text added: "ORANGE"

Commit message: Just about finished the layout
Parts:
- added TP1: TSV_RTN, Resistor_SMD:R_0805_2012Metric_Pad1.15x1.40mm_HandSolder, F.Cu at (120.3, 69.2)
- added TP10: SEG1_5V, TestPoint:TestPoint_Pad_D1.5mm, F.Cu at (50.8, 75.6)
- added TP11: SEG1_RTN, Resistor_SMD:R_0805_2012Metric_Pad1.15x1.40mm_HandSolder, F.Cu at (52.4, 63.5)
- added TP2: TSV_5V, TestPoint:TestPoint_Pad_D1.5mm, F.Cu at (116.2, 71.1)
- added TP3: SEG1_9V, TestPoint:TestPoint_Pad_D1.5mm, F.Cu at (104.8, 57.8)
- added TP4: LV_RTN, Resistor_SMD:R_0805_2012Metric_Pad1.15x1.40mm_HandSolder, F.Cu at (92.1, 141.0)
- added TP5: LV_5V, TestPoint:TestPoint_Pad_D1.5mm, F.Cu at (117.5, 137.2)
- added TP6: LV_24V, TestPoint:TestPoint_Pad_D1.5mm, F.Cu at (88.9, 101.0)
- added TP7: GLV_24V, TestPoint:TestPoint_Pad_D1.5mm, F.Cu at (102.2, 141.0)
- added TP8: SDA, TestPoint:TestPoint_Pad_D1.5mm, B.Cu at (130.2, 125.1)
- added TP9: SCL, TestPoint:TestPoint_Pad_D1.5mm, B.Cu at (130.2, 121.3)
- TP12, TP13: footprint TestPoint:TestPoint_Pad_D2.0mm -> TestPoint:TestPoint_Pad_D1.5mm
- TP14: footprint TestPoint:TestPoint_Pad_D2.0mm -> Resistor_SMD:R_0805_2012Metric_Pad1.15x1.40mm_HandSolder
- U3: footprint Package_TO_SOT_SMD:SOT-23-5_HandSoldering -> Package_TO_SOT_SMD:SOT-23-5
- moved LOGO1 132.3 mm to (179.7, 42.5)
- moved LOGO3 131.9 mm to (182.6, 59.7)
- moved LOGO2 131.5 mm to (195.6, 40.0)
- moved H1 31.9 mm to (123.2, 41.9)
- moved J12 18.3 mm to (97.8, 48.0)
- moved J16 18.3 mm to (90.6, 48.0)
- moved J11 16.7 mm to (114.3, 48.3)
- moved J15 16.7 mm to (107.3, 48.3)
- moved TP14 11.0 mm to (88.3, 53.7), turned to 90 degrees
- moved TP12 8.35 mm to (88.3, 57.8)
- moved C16 7.41 mm to (151.8, 57.8)
- moved R26 7.41 mm to (151.8, 68.6)
- moved U10 7.41 mm to (151.8, 64.8)
- moved U11 7.41 mm to (151.8, 61.0)
- moved H2 6.98 mm to (219.7, 42.5)
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Connections:
- C16 pad 2: /TSV_5V -> /SEG1_5V
- C17 pad 2: /SEG1_RTN -> /PACK_RTN
- C27 pad 1: /TSV_5V -> /SEG1_5V
- C28 pad 2: /SEG1_RTN -> /PACK_RTN
- J13 pad 1: /AIRS+ -> /AIRS-
- J13 pad 2: /AIRS- -> /AIRS+
- J14 pad 1: /AIRS+ -> /AIRS-
- J14 pad 2: /AIRS- -> /AIRS+
- J4 pad 1: /CHRG_DETECT+ -> /CHRG_DETECT-
- J4 pad 2: /CHRG_DETECT- -> /CHRG_DETECT+
- J5 pad 2: /SEG1_RTN -> /PACK_RTN
- J5 pad 5: /SEG1_RTN -> /PACK_RTN
- J8 pad 1: /AIRS+ -> /AIRS-
- J8 pad 2: /AIRS- -> /AIRS+
- J8 pad 5: /AIRS+ -> /AIRS-
- J8 pad 6: /AIRS- -> /AIRS+
- Q4 pad 3: /TSV_5V -> /SEG1_5V
- Q5 pad 3: /TSV_5V -> /SEG1_5V
- R28 pad 1: /TSV_5V -> /SEG1_5V
- R32 pad 1: /TSV_5V -> /SEG1_5V
- U11 pad 7: /TSV_5V -> /SEG1_5V
- U12 pad 6: /TSV_5V -> /SEG1_5V
- U14 pad 5: /SEG1_RTN -> /PACK_RTN
- U16 pad 7: /SEG1_RTN -> /PACK_RTN
Routing:
- net /SEG1_5V: track 2.12 -> 186.0 mm, vias 0 -> 5
- net /LV_3V3: track 129.9 -> 277.3 mm, vias 6 -> 15
- net /CHS_GND: track 5.50 -> 139.8 mm
- net /SCL_SEG1: track 0.00 -> 75.9 mm, vias 0 -> 3
- net /SDA_SEG1: track 0.00 -> 75.2 mm, vias 0 -> 1
- net /SEG1_9V: track 0.00 -> 66.8 mm, vias 0 -> 3
- net /MCU/~RESET: track 68.9 -> 114.9 mm, vias 5 -> 7
- net /SCL_GLV: track 119.7 -> 161.2 mm, vias 4 -> 6
- net /SDA_GLV: track 124.9 -> 163.7 mm, vias 4 -> 6
- net /GLV_24V: track 144.3 -> 175.5 mm
- net /TSV_VEHICLE+: track 0.00 -> 28.9 mm
- net /AIRS+: track 118.3 -> 143.6 mm
- net /GLV_RTN: track 60.3 -> 83.6 mm, vias 12 -> 19
- net /MCU/SLOOP_EN: track 8.83 -> 27.0 mm
- net /TSV_VEHICLE-: track 0.00 -> 17.4 mm
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- added copper zone on F.Cu, net (none)
- added copper zone on B.Cu, net /CHRG_IN+
- added copper zone on B.Cu, net /CHRG_IN-
- added copper zone on B.Cu, net /Charging/CurrentSensor+
- added copper zone on B.Cu, net /PACK+
- added copper zone on B.Cu, net /PACK-
- added copper zone on B.Cu, net /PACK_RTN
Other:
- board size 140.3 x 141.6 mm -> 139.7 x 117.5 mm
- board text added: "Accumulator Management System Fall 2019"
- board text added: "Bus Bar Current Sensor"
- board text added: "Low Voltage"
- board text added: "Made in USA"
- board text added: "PacMan v1.2 - Jon Abel"
- board text added: "TSV! High Voltage!"
